Commit message: urdf changes based on REP 103

File: src/aar2_description/urdf/aar2.urdf (robot description, URDF)
Before this commit: robot aar2, 7 links, 6 joints
Joints:
- joint base_front_left: origin xyz=-0.41 0.66 -0.35 rpy=0 -1.57 0 -> xyz=0.66 0.41 -0.35 rpy=-1.57 0 0
- joint base_front_right: origin xyz=0.41 0.66 -0.35 rpy=0 1.57 0 -> xyz=0.66 -0.41 -0.35 rpy=1.57 0 0
- joint base_mid_left: origin xyz=-0.41 0 -0.35 rpy=0 -1.57 0 -> xyz=0 0.41 -0.35 rpy=-1.57 0 0
- joint base_mid_right: origin xyz=0.41 0 -0.35 rpy=0 1.57 0 -> xyz=0 -0.41 -0.35 rpy=1.57 0 0
- joint base_rear_left: origin xyz=-0.41 -0.45 -0.35 rpy=0 -1.57 0 -> xyz=-0.45 0.41 -0.35 rpy=-1.57 0 0
- joint base_rear_right: origin xyz=0.41 -0.45 -0.35 rpy=0 1.57 0 -> xyz=-0.45 -0.41 -0.35 rpy=1.57 0 0

Commit message: add localization

File: src/aar2_description/urdf/aar2.urdf (robot description, URDF)
Before this commit: robot aar2, 7 links, 6 joints
Joints:
- joint base_front_left: axis 0 0 1 -> (none); type continuous -> fixed
- joint base_front_right: axis 0 0 -1 -> (none); type continuous -> fixed
- joint base_mid_left: axis 0 0 1 -> (none); type continuous -> fixed
- joint base_mid_right: axis 0 0 -1 -> (none); type continuous -> fixed
- joint base_rear_left: axis 0 0 1 -> (none); type continuous -> fixed
- joint base_rear_right: axis 0 0 -1 -> (none); type continuous -> fixed

Commit message: edit urdf, moved base link to centre of rotation

File: src/aar2_description/urdf/aar2.urdf (robot description, URDF)
Before this commit: robot aar2, 7 links, 6 joints
Joints:
- joint base_front_left: origin xyz=0.66 0.41 -0.35 rpy=-1.57 0 0 -> xyz=0.55 0.41 -0.35 rpy=-1.57 0 0
- joint base_front_right: origin xyz=0.66 -0.41 -0.35 rpy=1.57 0 0 -> xyz=0.55 -0.41 -0.35 rpy=1.57 0 0
- joint base_mid_left: origin xyz=0 0.41 -0.35 rpy=-1.57 0 0 -> xyz=-0.11 0.41 -0.35 rpy=-1.57 0 0
- joint base_mid_right: origin xyz=0 -0.41 -0.35 rpy=1.57 0 0 -> xyz=-0.11 -0.41 -0.35 rpy=1.57 0 0
- joint base_rear_left: origin xyz=-0.45 0.41 -0.35 rpy=-1.57 0 0 -> xyz=-0.55 0.41 -0.35 rpy=-1.57 0 0
- joint base_rear_right: origin xyz=-0.45 -0.41 -0.35 rpy=1.57 0 0 -> xyz=-0.55 -0.41 -0.35 rpy=1.57 0 0
