Commit message: fix urdf file

File: src/aar2_description/urdf/aar2test.urdf (robot description, URDF)
Before this commit: robot aar2, 7 links, 6 joints
Joints:
- joint base_front_left: origin xyz=0.55 0.41 -0.35 rpy=0 0 0 -> xyz=0.55 0.41 -0.35 rpy=-1.57 0 0
- joint base_front_right: origin xyz=0.55 -0.41 -0.35 rpy=0 0 0 -> xyz=0.55 -0.41 -0.35 rpy=1.57 0 0
- joint base_mid_left: origin xyz=-0.11 0.41 -0.35 rpy=0 0 0 -> xyz=-0.11 0.41 -0.35 rpy=-1.57 0 0
- joint base_mid_right: origin xyz=-0.11 -0.41 -0.35 rpy=0 0 0 -> xyz=-0.11 -0.41 -0.35 rpy=1.57 0 0
- joint base_rear_left: origin xyz=-0.55 0.41 -0.35 rpy=0 0 0 -> xyz=-0.55 0.41 -0.35 rpy=-1.57 0 0
- joint base_rear_right: origin xyz=-0.55 -0.41 -0.35 rpy=0 0 0 -> xyz=-0.55 -0.41 -0.35 rpy=1.57 0 0
