Commit message: changed teleop config and base node

File: src/aar2_description/urdf/aar2.urdf.xacro (robot description, xacro)
@@ -120,5 +120,5 @@
     <inertial>
       <mass value="0.001"/>
-      <origin xyz="0 0 0" rpy="0 0 0"/>
+      <origin xyz="0 0 0" rpy="-1.57 0 0"/>
       <inertia ixx="${dummy_inertia}" ixy="0.0" ixz="0.0" iyy="${dummy_inertia}" iyz="0.0" izz="${dummy_inertia}"/>
     </inertial>
@@ -127,5 +127,5 @@
     <parent link="chassis_link" />
     <child link="imu_link" />
-	<origin xyz="0 0 0" rpy="1.57 0 0" />
+	<origin xyz="0 0 0" rpy="0 0 0" />
   </joint>
   <!-- TODO: Same note as applies to imu_link -->
