Commit message: fixed 3 motor controller mode

File: aar2_description/urdf/aar2.urdf.xacro (robot description, xacro)
@@ -17,4 +17,5 @@
   <material name="yellow"><color rgba="0.8 0.8 0.0 1.0" /></material>
   <material name="black"><color rgba="0.15 0.15 0.15 1.0" /></material>
+  <material name="white"><color rgba="255 255 255 1.0" /></material>
   <xacro:macro name="wheel" params="prefix *joint_pose">
     <link name="${prefix}_wheel_link">
@@ -24,5 +25,5 @@
 		<cylinder length="${wheel_width}" radius="${wheel_radius}"/>
         </geometry>
-        <material name="black" />
+        <material name="white" />
       </visual>
       <collision>
@@ -81,5 +82,5 @@
         <box size ="${chassis_length} ${chassis_width} ${chassis_height}"/>
       </geometry>
-      <material name="dark_grey" />
+      <material name="yellow" />
     </visual>
     <collision>
